File: hardware/isolated_atlas0.sch (KiCad schematic (older format))
At the start: 15 parts, among them J201 CONN_01X02, P2 ATLAS_EC_PROBE, U201 ADM3260, U202 ATLAS_EC

Commit message: Cleanup footprints. Line up connectors on edges. Add second core port.
Parts:
- C201, C202, C203, C204, C205, C206: footprint Capacitors_SMD:C_0603_HandSoldering -> conservify:CAP-0603
- P2: footprint Oddities:Dummy_Empty -> conservify:Dummy_Empty
- R201, R202, R203, R204, R205: footprint Resistors_SMD:R_0603_HandSoldering -> conservify:RES-0603
Changed lines of the file:
@@
 EESchema Schematic File Version 2
-LIBS:power
-LIBS:device
-LIBS:transistors
-LIBS:conn
-LIBS:linear
-LIBS:regul
-LIBS:74xx
-LIBS:cmos4000
-LIBS:adc-dac
-LIBS:memory
-LIBS:xilinx
-LIBS:microcontrollers
-LIBS:dsp
-LIBS:microchip
-LIBS:analog_switches
-LIBS:motorola
-LIBS:intel
-LIBS:audio
-LIBS:interface
-LIBS:digital-audio
-LIBS:philips
-LIBS:display
-LIBS:cypress
-LIBS:siliconi
-LIBS:opto
-LIBS:atmel
-LIBS:contrib
-LIBS:valves
 LIBS:conservify
-LIBS:RocketScreamKicadLibrary
 LIBS:fk-atlas-cache
 EELAYER 25 0
@@
 F 0 "C203" H 5675 3900 50  0000 L CNN
 F 1 "0.1uF" H 5675 3700 50  0000 L CNN
-F 2 "Capacitors_SMD:C_0603_HandSoldering" H 5688 3650 50  0001 C CNN
+F 2 "conservify:CAP-0603" H 5688 3650 50  0001 C CNN
 F 3 "" H 5650 3800 50  0001 C CNN
 F 4 "0" H 5675 4000 50  0001 C CNN "price"
@@
 F 0 "C204" H 5675 4200 50  0000 L CNN
 F 1 "0.1uF" H 5675 4000 50  0000 L CNN
-F 2 "Capacitors_SMD:C_0603_HandSoldering" H 5688 3950 50  0001 C CNN
+F 2 "conservify:CAP-0603" H 5688 3950 50  0001 C CNN
 F 3 "" H 5650 4100 50  0001 C CNN
 F 4 "0" H 5675 4300 50  0001 C CNN "price"
@@
 F 0 "C205" H 5675 4500 50  0000 L CNN
 F 1 "10uF" H 5675 4300 50  0000 L CNN
-F 2 "Capacitors_SMD:C_0603_HandSoldering" H 5688 4250 50  0001 C CNN
+F 2 "conservify:CAP-0603" H 5688 4250 50  0001 C CNN
 F 3 "" H 5650 4400 50  0001 C CNN
 F 4 "0" H 5675 4600 50  0001 C CNN "price"
@@
 F 0 "C206" H 5675 4750 50  0000 L CNN
 F 1 "10uF" H 5675 4550 50  0000 L CNN
-F 2 "Capacitors_SMD:C_0603_HandSoldering" H 5688 4500 50  0001 C CNN
+F 2 "conservify:CAP-0603" H 5688 4500 50  0001 C CNN
 F 3 "" H 5650 4650 50  0001 C CNN
 F 4 "0" H 5675 4850 50  0001 C CNN "price"
@@
 F 0 "C201" H 2925 3900 50  0000 L CNN
 F 1 "0.1uF" H 2925 3700 50  0000 L CNN
-F 2 "Capacitors_SMD:C_0603_HandSoldering" H 2938 3650 50  0001 C CNN
+F 2 "conservify:CAP-0603" H 2938 3650 50  0001 C CNN
 F 3 "" H 2900 3800 50  0001 C CNN
 F 4 "0" H 2925 4000 50  0001 C CNN "price"
@@
 F 0 "C202" H 2925 4200 50  0000 L CNN
 F 1 "10uF" H 2925 4000 50  0000 L CNN
-F 2 "Capacitors_SMD:C_0603_HandSoldering" H 2938 3950 50  0001 C CNN
+F 2 "conservify:CAP-0603" H 2938 3950 50  0001 C CNN
 F 3 "" H 2900 4100 50  0001 C CNN
 F 4 "0" H 2925 4300 50  0001 C CNN "price"
@@
 F 0 "R201" V 5730 3300 50  0000 C CNN
 F 1 "1.5K" V 5650 3300 50  0000 C CNN
-F 2 "Resistors_SMD:R_0603_HandSoldering" V 5580 3300 50  0001 C CNN
+F 2 "conservify:RES-0603" V 5580 3300 50  0001 C CNN
 F 3 "" H 5650 3300 50  0001 C CNN
 F 4 "0" H 5730 3400 50  0001 C CNN "price"
@@
 F 0 "R202" V 6330 2700 50  0000 C CNN
 F 1 "1.5K" V 6250 2700 50  0000 C CNN
-F 2 "Resistors_SMD:R_0603_HandSoldering" V 6180 2700 50  0001 C CNN
+F 2 "conservify:RES-0603" V 6180 2700 50  0001 C CNN
 F 3 "" H 6250 2700 50  0001 C CNN
 F 4 "0" H 6330 2800 50  0001 C CNN "price"
@@
 F 0 "R204" V 6780 2700 50  0000 C CNN
 F 1 "1.5K" V 6700 2700 50  0000 C CNN
-F 2 "Resistors_SMD:R_0603_HandSoldering" V 6630 2700 50  0001 C CNN
+F 2 "conservify:RES-0603" V 6630 2700 50  0001 C CNN
 F 3 "" H 6700 2700 50  0001 C CNN
 F 4 "0" H 6780 2800 50  0001 C CNN "price"
@@
 F 0 "R203" V 6380 3250 50  0000 C CNN
 F 1 "4.7K" V 6300 3250 50  0000 C CNN
-F 2 "Resistors_SMD:R_0603_HandSoldering" V 6230 3250 50  0001 C CNN
+F 2 "conservify:RES-0603" V 6230 3250 50  0001 C CNN
 F 3 "" H 6300 3250 50  0001 C CNN
 F 4 "0" H 6380 3350 50  0001 C CNN "price"
@@
 F 0 "R205" V 6880 3250 50  0000 C CNN
 F 1 "4.7K" V 6800 3250 50  0000 C CNN
-F 2 "Resistors_SMD:R_0603_HandSoldering" V 6730 3250 50  0001 C CNN
+F 2 "conservify:RES-0603" V 6730 3250 50  0001 C CNN
 F 3 "" H 6800 3250 50  0001 C CNN
 F 4 "0" H 6880 3350 50  0001 C CNN "price"
@@
 $EndComp
 $Comp
-L VCC #PWR64
+L VCC #PWR58
 U 1 1 594C2D26
 P 2450 3750
-F 0 "#PWR64" H 2450 3600 50  0001 C CNN
+F 0 "#PWR58" H 2450 3600 50  0001 C CNN
 F 1 "VCC" H 2450 3900 50  0000 C CNN
 F 2 "" H 2450 3750 50  0001 C CNN
@@
 $EndComp
 $Comp
-L VCC #PWR63
+L VCC #PWR57
 U 1 1 594C2D28
 P 2450 2350
-F 0 "#PWR63" H 2450 2200 50  0001 C CNN
+F 0 "#PWR57" H 2450 2200 50  0001 C CNN
 F 1 "VCC" H 2450 2500 50  0000 C CNN
 F 2 "" H 2450 2350 50  0001 C CNN
@@
 F 0 "P2" H 8800 3550 60  0000 C CNN
 F 1 "ATLAS_EC_PROBE" H 8800 3450 60  0000 C CNN
-F 2 "Oddities:Dummy_Empty" H 8800 3550 60  0001 C CNN
+F 2 "conservify:Dummy_Empty" H 8800 3550 60  0001 C CNN
 F 3 "" H 8800 3550 60  0001 C CNN
 	1    8800 3550
