File: hardware/fk-atlas.sch (KiCad schematic (older format))
At the start: 56 parts, among them J1 CONN-HDR-2x5, J2 MICRO-USB, J3 Conn_01x02, J4 CONN_01x03_SERIAL, J5 Conn_01x05, J6 CONN_01x04, J7 Conn_01x05, M1 MOUNT_HOLE, M2 MOUNT_HOLE, M3 MOUNT_HOLE, M4 MOUNT_HOLE, M5 FIDUCIAL, M6 FIDUCIAL, M7 FIDUCIAL, Q4 2N7002LT1G, SW1 SPNO, U1 S25FL1xxK0XM, U2 ATSAMD21G18A-AU, U3 MCP1700T-3302E/MB, U4 TPS2051B, U5 SK6812, Y1 FC-135

Commit message: Consistent part values across our schematics.
Parts:
- C1, C10, C12: value 4.7uF 10V X5R -> 4.7uF
- C11: value 1uF 50V X5R -> 1uF
- C13: value 4.7nF 25V X7R -> 4.7nF
- C14, C15, C6: value 1uF 10V X5R -> 1uF
- D6: value DIODE_DUAL_Schottky -> PMEG3020CPA
- U1: value S25FL1xxK0XM -> S25FL116K0XMFI041

Commit message: Part updates.
Parts:
- C1, C10, C12: Critical (none) -> (none); MFN (none) -> AVX; MFP (none) -> 0603ZD475MAT2A; Notes (none) -> (none); Package (none) -> (none); Source (none) -> ANY; Subsystem (none) -> (none)
- C11: Critical (none) -> (none); MFN (none) -> Taiyo Yuden; MFP (none) -> UMK107BJ105KA-T; Notes (none) -> (none); Package (none) -> (none); Source (none) -> ANY; Subsystem (none) -> (none)
- C13: Critical (none) -> (none); MFN (none) -> KEMET; MFP (none) -> C0603C472K9RACTU; Notes (none) -> (none); Package (none) -> (none); Source (none) -> ANY; Subsystem (none) -> (none); spn1 603-AC603KRX7R8BB472 -> 80-C0603C472K9R
- C14, C15, C6: Critical (none) -> (none); MFN (none) -> Taiyo Yuden; MFP (none) -> UMK107BJ105KA-T; Notes (none) -> (none); Package (none) -> (none); Source (none) -> ANY; Subsystem (none) -> (none); spn1 581-0603YD105K -> 963-UMK107BJ105KA-T
- C16, C17, C18, C2, C5, C7, C8, C9: Critical (none) -> (none); MFN (none) -> Murata Electronics; MFP (none) -> GRM188R71H104KA93D; Notes (none) -> (none); Package (none) -> (none); Source (none) -> ANY; Subsystem (none) -> (none)
- C19: Critical (none) -> (none); MFN (none) -> Taiyo Yuden; MFP (none) -> LMK107BBJ106KALT; Notes (none) -> (none); Package (none) -> (none); SPN1 (none) -> 963-LMK107BBJ106KALT; Source (none) -> ANY; Subsystem (none) -> (none); Supplier1 (none) -> mouser
- C3, C4: Critical (none) -> (none); MFN (none) -> AVX; MFP (none) -> 06035A180JAT2A; Notes (none) -> (none); Package (none) -> (none); Source (none) -> ANY; Subsystem (none) -> (none)
- D4: Critical (none) -> (none); MFN (none) -> Lite-On; MFP (none) -> LTST-C190KFKT; Notes (none) -> (none); Package (none) -> (none); Source (none) -> ANY; Subsystem (none) -> (none)
- D5: Critical (none) -> (none); MFN (none) -> Nexperia; MFP (none) -> PRTR5V0U2X,215; Notes (none) -> (none); Package (none) -> (none); Source (none) -> ANY; Subsystem (none) -> (none)
- D6: Critical (none) -> (none); MFN (none) -> Nexperia; MFP (none) -> PMEG3020CPA,115; Notes (none) -> (none); Package (none) -> (none); SPN1 (none) -> 771-PMEG3020CPA115; Source (none) -> ANY; Subsystem (none) -> (none); Supplier1 (none) -> mouser
- F1: Critical (none) -> (none); MFN (none) -> Bourns; MFP (none) -> MF-PSMF050X-2; Notes (none) -> (none); Package (none) -> (none); Source (none) -> ANY; Subsystem (none) -> (none)
- J1: value CONN-HDR-2x5 -> CONN_02x05_SWD; Critical (none) -> (none); MFN (none) -> Amphenol FCI; MFP (none) -> 20021121-00010C4LF; Notes (none) -> (none); Package (none) -> (none); Source (none) -> ANY; Subsystem (none) -> (none)
- J2: Critical (none) -> (none); MFN (none) -> Hirose Connector; MFP (none) -> ZX62D-B-5PA8(30); Notes (none) -> (none); Package (none) -> (none); Source (none) -> ANY; Subsystem (none) -> (none)
- J3, J6, M1, M2, M3, M4, M5, M6, M7, U4: Critical (none) -> (none); MFN (none) -> (none); MFP (none) -> (none); Notes (none) -> (none); Package (none) -> (none); SPN1 (none) -> (none); Source (none) -> ANY; Subsystem (none) -> (none); Supplier1 (none) -> (none)
- J4: Critical (none) -> (none); MFN (none) -> Molex; MFP (none) -> 502382-0370; Notes (none) -> (none); Package (none) -> (none); SPN1 (none) -> 538-502382-0370; Source (none) -> ANY; Subsystem (none) -> (none); Supplier1 (none) -> mouser
- J5, J7: Critical (none) -> (none); MFN (none) -> Molex; MFP (none) -> 502382-0570; Notes (none) -> (none); Package (none) -> (none); SPN1 (none) -> 538-502382-0570; Source (none) -> ANY; Subsystem (none) -> (none); Supplier1 (none) -> mouser
- L1, L2: Critical (none) -> (none); MFN (none) -> Murata Electronics; MFP (none) -> BLM18KG221SN1D; Notes (none) -> (none); Package (none) -> (none); Source (none) -> ANY; Subsystem (none) -> (none)
- Q4: Critical (none) -> (none); MFN (none) -> ON Semiconductor; MFP (none) -> 2N7002LT1G; Notes (none) -> (none); Package (none) -> (none); Source (none) -> ANY; Subsystem (none) -> (none)
- R1, R12: Critical (none) -> (none); MFN (none) -> Yageo; MFP (none) -> RC0603FR-0710KL; Notes (none) -> (none); Package (none) -> (none); Source (none) -> ANY; Subsystem (none) -> (none)
- R10: Critical (none) -> (none); MFN (none) -> Yageo; MFP (none) -> RC0603FR-071ML; Notes (none) -> (none); Package (none) -> (none); Source (none) -> ANY; Subsystem (none) -> (none)
- R11: Critical (none) -> (none); MFN (none) -> Yageo; MFP (none) -> RC0603FR-072K2L; Notes (none) -> (none); Package (none) -> (none); Source (none) -> ANY; Subsystem (none) -> (none)
- R2, R9: Critical (none) -> (none); MFN (none) -> Yageo; MFP (none) -> RC0603FR-07330RL; Notes (none) -> (none); Package (none) -> (none); Source (none) -> ANY; Subsystem (none) -> (none)
- R4, R5: Critical (none) -> (none); MFN (none) -> Yageo; MFP (none) -> AF0603JR-074K7L; Notes (none) -> (none); Package (none) -> (none); Source (none) -> ANY; Subsystem (none) -> (none); Supplier1 (none) -> mouser
- R8: Critical (none) -> (none); MFN (none) -> Yageo; MFP (none) -> RC0603FR-07100KL; Notes (none) -> (none); Package (none) -> (none); Source (none) -> ANY; Subsystem (none) -> (none)
- SW1: Critical (none) -> (none); MFN (none) -> Wurth Electronics; MFP (none) -> 434331045822; Notes (none) -> (none); Package (none) -> (none); Source (none) -> ANY; Subsystem (none) -> (none)
- U1: Critical (none) -> (none); MFN (none) -> Cypress Semiconductor; MFP (none) -> S25FL116K0XMFI041; Notes (none) -> (none); Package (none) -> (none); Source (none) -> ANY; Subsystem (none) -> (none); Supplier1 (none) -> mouser
- U2: Critical (none) -> (none); MFN (none) -> Microchip Technology / Atmel; MFP (none) -> ATSAMD21G18A-AU; Notes (none) -> (none); Package (none) -> (none); Source (none) -> ANY; Subsystem (none) -> (none)
- U3: Critical (none) -> (none); MFN (none) -> Microchip Technology; MFP (none) -> MCP1700T-3302E/MB; Notes (none) -> (none); Package (none) -> (none); Source (none) -> ANY; Subsystem (none) -> (none)
- U5: Critical (none) -> (none); MFN (none) -> Adafruit; MFP (none) -> 1655; Notes (none) -> (none); Package (none) -> (none); SPN1 (none) -> 1528-1104-ND; Source (none) -> ANY; Subsystem (none) -> (none); Supplier1 (none) -> digikey
- Y1: Critical (none) -> (none); MFN (none) -> Epson Timing; MFP (none) -> FC-135 32.7680KA-A3; Notes (none) -> (none); Package (none) -> (none); Source (none) -> ANY; Subsystem (none) -> (none)

Commit message: Fix Sk6812 and include pins in signal names.
Connections:
- net labels added: D12_PERIPH_EN, D5_FLASH_CS
- net labels removed: FLASH_CS, PERIPH_EN, PRESSURE

Commit message: Fix DRC in schematic mode.
Parts:
- C1, C10, C11, C12, C13, C14, C15, C16, C17, C18, C19, C2, C3, C4, C5, C6, C7, C8, C9: symbol fk-atlas-rescue:CAPACITOR-CERAMIC -> conservify:CAPACITOR_CERAMIC
- D4: symbol fk-atlas-rescue:LED-SINGLE -> conservify:LED_SINGLE
- D6: symbol fk-atlas-rescue:DIODE_DUAL_Schottky -> conservify:DIODE_DUAL_SCHOTTKY
- J1: symbol fk-atlas-rescue:CONN-HDR-2x5 -> conservify:CONN_02x05_SWD
- J2: symbol fk-atlas-rescue:MICRO-USB -> conservify:MICRO_USB
- J3: symbol fk-atlas-rescue:Conn_01x02 -> conservify:CONN_01x02
- J5, J7: symbol fk-atlas-rescue:Conn_01x05 -> conservify:CONN_01x05
- Q4: symbol fk-atlas-rescue:MOSFET-N -> conservify:MOSFET_N
- R4, R5: symbol fk-atlas-rescue:R -> conservify:RESISTOR
- SW1: symbol fk-atlas-rescue:TACT-SWITCH_2Pins -> conservify:SWITCH_CONN_02
- U2: symbol fk-atlas-rescue:ATSAMD21G18A-AU -> conservify:ATSAMD21G18A_AU
Connections:
- net labels removed: AREF
- wire segments 266 -> 270
- no-connect marks 6 -> 26
Other:
- moved on the sheet: M5, M6, M7

Commit message: Use more compatible FP for flash.
Parts:
- U1: footprint conservify:SOIC-8-N -> conservify:SOIC-8-N-WIDE
Changed lines of the file:
@@
 F 0 "U1" H 2200 9450 60  0000 C CNN
 F 1 "S25FL116K0XMFI041" H 2200 8850 60  0000 C CNN
-F 2 "conservify:SOIC-8-N" H 2200 8750 60  0001 C CNN
+F 2 "conservify:SOIC-8-N-WIDE" H 2200 8750 60  0001 C CNN
 F 3 "" H 2000 9200 60  0000 C CNN
 F 4 " " H 2200 9550 50  0001 C CNN "Critical"

Commit message: Consistency in part values
Parts:
- J3: value Conn_01x02 -> CONN_01x02
- J5, J7: value Conn_01x05 -> CONN_01x05
- J6: MFN (none) -> Molex; MFP (none) -> 502382-0470; SPN1 (none) -> WM4781CT-ND; Supplier1 (none) -> digikey
- U4: MFN (none) -> Texas Instruments; MFP (none) -> TPS2051BDBVR; SPN1 (none) -> 296-21265-1-ND; Supplier1 (none) -> digikey

Commit message: Separate power control for Atlas from Flash. Add pull downs.
Parts:
- removed U4: TPS2051B, conservify:SOT-23-5_HandSoldering, symbol conservify:TPS2051B
- added C20: 100nF, conservify:CAP-0603, symbol conservify:CAPACITOR_CERAMIC
- added C21: 10uF, conservify:CAP-0603, symbol conservify:CAPACITOR_CERAMIC
- added J8: CONN_01x02, conservify:SJ_OPEN, symbol conservify:CONN_01x02
- added R3, R6, R7: 10K, conservify:RES-0603, symbol conservify:RESISTOR
- added U4: TPS2052B, conservify:SOIC-8-N, symbol conservify:TPS2052B
Connections:
- net labels added: ATLAS_3V3, D6_ATLAS_EN
- net labels removed: D6
- wire segments 270 -> 282
- no-connect marks 26 -> 25
Other:
- moved on the sheet: C18, C19, J3, R12
