File: hardware/isolated_atlas2.sch (KiCad schematic (older format))
At the start: 15 parts, among them J401 CONN_01X02, P4 ATLAS_PH_PROBE, U401 ADM3260, U402 ATLAS_PH

Commit message: Consistent part values across our schematics.
Parts:
- C401, C403, C404: value 0.1uF -> 100nF

Commit message: Part updates.
Parts:
- C401, C403, C404: Critical (none) -> (none); MFN (none) -> Murata Electronics; MFP (none) -> GRM188R71H104KA93D; Notes (none) -> (none); Package (none) -> (none); Source (none) -> ANY; Subsystem (none) -> (none); Supplier1 (none) -> mouser
- C402, C405, C406: Critical (none) -> (none); MFN (none) -> Taiyo Yuden; MFP (none) -> LMK107BBJ106KALT; Notes (none) -> (none); Package (none) -> (none); Source (none) -> ANY; Subsystem (none) -> (none); Supplier1 (none) -> mouser; spn1 81-GRM188R60J106ME47 -> 963-LMK107BBJ106KALT
- J401: Critical (none) -> (none); MFN (none) -> Amphenol RF; MFP (none) -> 031-5431; Notes (none) -> (none); Package (none) -> (none); Source (none) -> ANY; Subsystem (none) -> (none); Supplier1 (none) -> mouser
- P4: Critical (none) -> (none); MFN (none) -> (none); MFP (none) -> (none); Notes (none) -> (none); Package (none) -> (none); SPN1 (none) -> (none); Source (none) -> ANY; Subsystem (none) -> (none); Supplier1 (none) -> (none)
- R401, R402, R404: Critical (none) -> (none); MFN (none) -> (none); MFP (none) -> (none); Notes (none) -> (none); Package (none) -> (none); Source (none) -> ANY; Subsystem (none) -> (none); Supplier1 (none) -> (none)
- R403, R405: Critical (none) -> (none); MFN (none) -> Yageo; MFP (none) -> AF0603JR-074K7L; Notes (none) -> (none); Package (none) -> (none); Source (none) -> ANY; Subsystem (none) -> (none); Supplier1 (none) -> mouser
- U401: Critical (none) -> (none); MFN (none) -> Analog Devices / Linear Technology; MFP (none) -> ADM3260ARSZ; Notes (none) -> (none); Package (none) -> (none); Source (none) -> ANY; Subsystem (none) -> (none); Supplier1 (none) -> mouser
- U402: Critical (none) -> (none); MFN (none) -> (none); MFP (none) -> (none); Notes (none) -> (none); Package (none) -> (none); SPN1 (none) -> (none); Source (none) -> ANY; Subsystem (none) -> (none); Supplier1 (none) -> atlas

Commit message: Fix DRC in schematic mode.
Parts:
- C401, C402, C403, C404, C405, C406: symbol fk-atlas-rescue:C -> conservify:CAPACITOR_CERAMIC
- J401: symbol fk-atlas-rescue:CONN_01X02 -> conservify:CONN_01x02
- P4: symbol fk-atlas-rescue:WATER_PROBE -> conservify:ATLAS_WATER_PROBE
- R401, R402, R403, R404, R405: symbol fk-atlas-rescue:R -> conservify:R
- U401: symbol fk-atlas-rescue:adm3260 -> conservify:ADM3260
Connections:
- wire segments 52 -> 78
Changed lines of the file:
@@
 $EndDescr
 $Comp
-L fk-atlas-rescue:adm3260 U401
+L conservify:ADM3260 U401
 U 1 1 594C2CF1
 P 4400 2900
@@
 $EndComp
 $Comp
-L fk-atlas-rescue:C C403
+L conservify:CAPACITOR_CERAMIC C403
 U 1 1 594C2CF4
 P 5650 3800
@@
 $EndComp
 $Comp
-L fk-atlas-rescue:C C404
+L conservify:CAPACITOR_CERAMIC C404
 U 1 1 594C2CF8
 P 5650 4100
@@
 $EndComp
 $Comp
-L fk-atlas-rescue:C C405
+L conservify:CAPACITOR_CERAMIC C405
 U 1 1 594C2CFB
 P 5650 4400
@@
 $EndComp
 $Comp
-L fk-atlas-rescue:C C406
+L conservify:CAPACITOR_CERAMIC C406
 U 1 1 594C2CFF
 P 5650 4650
@@
 $EndComp
 $Comp
-L fk-atlas-rescue:C C401
+L conservify:CAPACITOR_CERAMIC C401
 U 1 1 594C2D03
 P 2900 3800
@@
 $EndComp
 $Comp
-L fk-atlas-rescue:C C402
+L conservify:CAPACITOR_CERAMIC C402
 U 1 1 594C2D07
 P 2900 4100
@@
 $EndComp
 $Comp
-L fk-atlas-rescue:R R401
+L conservify:R R401
 U 1 1 594C2D0B
 P 5650 3300
@@
 $EndComp
 $Comp
-L fk-atlas-rescue:R R402
+L conservify:R R402
 U 1 1 594C2D10
 P 6250 2700
@@
 $EndComp
 $Comp
-L fk-atlas-rescue:R R404
+L conservify:R R404
 U 1 1 594C2D14
 P 6700 2700
@@
 $EndComp
 $Comp
-L fk-atlas-rescue:R R403
+L conservify:R R403
 U 1 1 5948E450
 P 6300 3250
@@
 $EndComp
 $Comp
-L fk-atlas-rescue:R R405
+L conservify:R R405
 U 1 1 594C2D1B
 P 6800 3250
@@
 $EndComp
 $Comp
-L fk-atlas-rescue:VCC #PWR061
+L conservify:VCC #PWR061
 U 1 1 594C2D24
 P 2450 3750
@@
 $EndComp
 $Comp
-L fk-atlas-rescue:VCC #PWR062
+L conservify:VCC #PWR062
 U 1 1 594C2D2A
 P 2450 2350
@@
 $EndComp
 $Comp
-L fk-atlas-rescue:CONN_01X02 J401
+L conservify:CONN_01x02 J401
 U 1 1 59A1BC7D
-P 10100 2950
-F 0 "J401" H 10100 3100 50  0000 C CNN
-F 1 "CONN_01X02" V 10200 2950 50  0000 C CNN
-F 2 "conservify:BNC" H 10100 2950 50  0001 C CNN
-F 3 "" H 10100 2950 50  0001 C CNN
-F 4 " " H 10100 3200 50  0001 C CNN "Critical"
-F 5 "Amphenol RF" H 10100 3200 50  0001 C CNN "MFN"
-F 6 "031-5431" H 10100 3200 50  0001 C CNN "MFP"
-F 7 " " H 10100 3200 50  0001 C CNN "Notes"
-F 8 " " H 10100 3200 50  0001 C CNN "Package"
-F 9 "ANY" H 10100 3200 50  0001 C CNN "Source"
-F 10 " " H 10100 3200 50  0001 C CNN "Subsystem"
-F 11 "mouser" H 10100 3200 50  0001 C CNN "Supplier1"
-F 12 "0" H 10100 3200 50  0001 C CNN "price"
-F 13 "523-31-5431" H 250 0   50  0001 C CNN "spn1"
-	1    10100 2950
-	1    0    0    -1
-$EndComp
-$Comp
-L fk-atlas-rescue:WATER_PROBE P4
+P 10100 2900
+F 0 "J401" H 10100 3050 50  0000 C CNN
+F 1 "CONN_01X02" V 10200 2900 50  0000 C CNN
+F 2 "conservify:BNC" H 10100 2900 50  0001 C CNN
+F 3 "" H 10100 2900 50  0001 C CNN
+F 4 " " H 10100 3150 50  0001 C CNN "Critical"
+F 5 "Amphenol RF" H 10100 3150 50  0001 C CNN "MFN"
+F 6 "031-5431" H 10100 3150 50  0001 C CNN "MFP"
+F 7 " " H 10100 3150 50  0001 C CNN "Notes"
+F 8 " " H 10100 3150 50  0001 C CNN "Package"
+F 9 "ANY" H 10100 3150 50  0001 C CNN "Source"
+F 10 " " H 10100 3150 50  0001 C CNN "Subsystem"
+F 11 "mouser" H 10100 3150 50  0001 C CNN "Supplier1"
+F 12 "0" H 10100 3150 50  0001 C CNN "price"
+F 13 "523-31-5431" H 250 -50 50  0001 C CNN "spn1"
+	1    10100 2900
+	1    0    0    -1
+$EndComp
+$Comp
+L conservify:ATLAS_WATER_PROBE P4
 U 1 1 59D2A29B
 P 8800 3600
@@
 F 12 " " H 8800 3700 50  0001 C CNN "Supplier1"
 	1    8800 3600
+	1    0    0    -1
+$EndComp
+$Comp
+L conservify:PWR_FLAG #FLG0107
+U 1 1 5BCC2A39
+P 7400 4900
+F 0 "#FLG0107" H 7400 4975 50  0001 C CNN
+F 1 "PWR_FLAG" H 7400 5050 50  0000 C CNN
+F 2 "" H 7400 4900 50  0001 C CNN
+F 3 "~" H 7400 4900 50  0001 C CNN
+	1    7400 4900
 	1    0    0    -1
 $EndComp
@@
 PH_PGND
 Wire Wire Line
-	5200 3300 5500 3300
-Wire Wire Line
-	5350 3300 5350 5000
+	5200 3300 5350 3300
+Wire Wire Line
+	5350 3300 5350 3400
 Wire Wire Line
 	5350 3600 5200 3600
@@
 	5800 3800 6000 3800
 Wire Wire Line
-	6000 3600 6000 4650
+	6000 3600 6000 3800
 Wire Wire Line
 	6000 4650 5800 4650
@@
 	5800 4100 6000 4100
 Wire Wire Line
-	5200 2800 7800 2800
-Wire Wire Line
-	5200 2900 7800 2900
-Wire Wire Line
-	5200 2700 6100 2700
+	5200 2800 6300 2800
+Wire Wire Line
+	5200 2900 6800 2900
+Wire Wire Line
+	5200 2700 6000 2700
 Wire Wire Line
 	6000 2700 6000 3300
@@
 	5350 2600 5350 2500
 Wire Wire Line
-	5200 2500 7400 2500
+	5200 2500 5350 2500
 Wire Wire Line
 	6900 2500 6900 2700
@@
 	6300 3400 6300 3600
 Wire Wire Line
-	6000 3600 6800 3600
+	6000 3600 6300 3600
 Wire Wire Line
 	6800 3600 6800 3400
 Wire Wire Line
-	2450 2600 3650 2600
-Wire Wire Line
-	2450 2350 2450 2600
+	2450 2600 3500 2600
+Wire Wire Line
+	2450 2350 2450 2450
 Wire Wire Line
 	3650 2500 3500 2500
@@
 	3650 3200 3050 3200
 Wire Wire Line
-	3050 3200 3050 4250
+	3050 3200 3050 3300
 Wire Wire Line
 	3050 4250 1750 4250
@@
 Wire Wire Line
 	9450 3000 9900 3000
+Wire Wire Line
+	7400 4900 7400 5000
+Wire Wire Line
+	5350 3500 5350 3600
+Wire Wire Line
+	5350 3400 5350 3500
+Wire Wire Line
+	5350 3600 5350 3800
+Wire Wire Line
+	5350 4400 5350 4650
+Wire Wire Line
+	5350 4100 5350 4400
+Wire Wire Line
+	5350 3800 5350 4100
+Wire Wire Line
+	6000 4400 6000 4650
+Wire Wire Line
+	6000 4100 6000 4400
+Wire Wire Line
+	5350 3300 5500 3300
+Wire Wire Line
+	5350 2500 6900 2500
+Wire Wire Line
+	6000 2700 6100 2700
+Wire Wire Line
+	6300 2800 7800 2800
+Wire Wire Line
+	6800 2900 7800 2900
+Wire Wire Line
+	3500 2600 3650 2600
+Wire Wire Line
+	3050 3800 3050 4100
+Wire Wire Line
+	3050 4100 3050 4250
+Wire Wire Line
+	3050 3600 3050 3800
+Wire Wire Line
+	3050 3500 3050 3600
+Wire Wire Line
+	3050 3400 3050 3500
+Wire Wire Line
+	3050 3300 3050 3400
+Wire Wire Line
+	2450 2450 2450 2600
+Wire Wire Line
+	5350 4650 5350 5000
+Wire Wire Line
+	6300 3600 6800 3600
+Wire Wire Line
+	6000 3800 6000 4100
+Wire Wire Line
+	6900 2500 7400 2500
 Connection ~ 5350 3500
 Connection ~ 5350 3400
@@
 Connection ~ 6300 3600
 Connection ~ 6000 3800
-Connection ~ 3050 4250
 Connection ~ 6900 2500
 NoConn ~ 3650 3000

Commit message: Drop prototype Atlas modules - focus on getting OEM boards working.
Parts:
- U402: footprint conservify:ATLAS_SENSOR_BOARD_COMBO -> conservify:ATLAS_SENSOR_BOARD_OEM
Changed lines of the file:
@@
 F 0 "U402" H 8100 2550 60  0000 C CNN
 F 1 "ATLAS_PH" H 8600 2850 60  0000 C CNN
-F 2 "conservify:ATLAS_SENSOR_BOARD_COMBO" H 8550 2900 60  0001 C CNN
+F 2 "conservify:ATLAS_SENSOR_BOARD_OEM" H 8550 2900 60  0001 C CNN
 F 3 "" H 8550 2900 60  0001 C CNN
 F 4 " " H 8100 2650 50  0001 C CNN "Critical"

Commit message: Trying out some test points.
Parts:
- added J13, J14: CONN_01x02, conservify:TP_Pads_D1.5mm_1x2, symbol conservify:CONN_01x02
Connections:
- wire segments 78 -> 82
Changed lines of the file:
@@
 NoConn ~ 3650 3000
 NoConn ~ 5200 3000
+Text Label 8350 4500 0    60   ~ 0
+ISO_GND
+Text Label 8350 4400 0    60   ~ 0
+ISO_VCC
+Text Label 8350 4150 0    60   ~ 0
+ISO_SCL
+Text Label 8350 4250 0    60   ~ 0
+ISO_SDA
+Wire Wire Line
+	8350 4150 8750 4150
+Wire Wire Line
+	8750 4250 8350 4250
+Wire Wire Line
+	8350 4400 8750 4400
+Wire Wire Line
+	8750 4500 8350 4500
+$Comp
+L conservify:CONN_01x02 J?
+U 1 1 5C0ECD1F
+P 8950 4150
+AR Path="/594C282A/5C0ECD1F" Ref="J?"  Part="1"
+AR Path="/594C282D/5C0ECD1F" Ref="J13"  Part="1"
+F 0 "J13" H 9029 4142 50  0000 L CNN
+F 1 "CONN_01x02" H 9029 4051 50  0000 L CNN
+F 2 "conservify:TP_Pads_D1.5mm_1x2" H 8950 4150 50  0001 C CNN
+F 3 "" H 8950 4150 50  0001 C CNN
+	1    8950 4150
+	1    0    0    -1
+$EndComp
+$Comp
+L conservify:CONN_01x02 J?
+U 1 1 5C0ECD26
+P 8950 4400
+AR Path="/594C282A/5C0ECD26" Ref="J?"  Part="1"
+AR Path="/594C282D/5C0ECD26" Ref="J14"  Part="1"
+F 0 "J14" H 9029 4392 50  0000 L CNN
+F 1 "CONN_01x02" H 9029 4301 50  0000 L CNN
+F 2 "conservify:TP_Pads_D1.5mm_1x2" H 8950 4400 50  0001 C CNN
+F 3 "" H 8950 4400 50  0001 C CNN
+	1    8950 4400
+	1    0    0    -1
+$EndComp
 $EndSCHEMATC
